File: kicad/tesi.kicad_pcb (KiCad board)
At the start: 2 copper layers, 100 x 100 mm, 30 parts, among them SW1 POWER, U1 MAX4466, U2 MPR121, U3 BNO055, U4 VL53L1CX

Commit message: updates
Parts:
- removed LiPo Battery: Battery, Library:Lipo Battery 400 mAh
- added BT1: LIPO BATTERY, tesi:Lipo Battery 500 mAh - 38x30.5mm, F.Cu at (129.2, 85.8)
- added RV1: POT, Potentiometer_THT:Potentiometer_TT_P0915N, F.Cu at (56.5, 77.8)
- A2: value Adafruit Feather HUZZAH32 -> ESP32
- B1: value MUTE -> ~
- H5, H6: footprint MountingHole:MountingHole_4mm -> tesi:MountingHole_3.2mm_M3
- TP1, TP2, TP3, TP4, TP5, TP6, TP7, TP8: footprint TestPoint:TestPoint_Pad_D4.0mm -> tesi:TouchPad - 4.0mm
- U2: value MPR121 -> BNO055; footprint tesi:MPR121 -> tesi:BNO055
- U3: value BNO055 -> MPR121; footprint tesi:BNO055 -> tesi:MPR121
- moved TP8 76.2 mm to (137.7, 140.8)
- moved TP7 75.0 mm to (126.5, 141.0)
- moved TP6 73.7 mm to (115.3, 141.0)
- moved TP5 72.4 mm to (104.1, 141.0)
- moved SW1 63.4 mm to (78.3, 60.0), turned to 180 degrees
- moved U4 62.8 mm to (119.4, 112.3)
- moved H5 59.4 mm to (113.8, 87.9)
- moved U3 56.3 mm to (114.4, 128.8), turned to 180 degrees
- moved B1 54.1 mm to (79.6, 75.7), turned to 180 degrees
- moved TP1 53.4 mm to (59.2, 140.9), turned to 180 degrees
- moved H6 47.4 mm to (144.3, 88.0)
- moved R5 40.1 mm to (129.1, 62.8)
- moved D1 39.9 mm to (135.3, 62.2), turned to 90 degrees
- moved R2 37.8 mm to (80.1, 91.4), turned to 180 degrees
- moved R1 34.3 mm to (75.0, 85.5)
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- renumbered R7 to R6, R6 to R7
Connections:
- A2 pad 20: Net-(A2-A7/IO32) -> unconnected-(A2-A7/IO32-Pad20)
- A2 pad 6: unconnected-(A2-DAC1/A1-Pad6) -> Net-(A2-DAC1/A1)
- A2 pad 8: unconnected-(A2-I39/A3-Pad8) -> Net-(A2-I39/A3)
- B1 pad 2: Net-(A2-A7/IO32) -> Net-(A2-DAC1/A1)
- R1 pad 1: Net-(A2-I34/A2) -> Net-(A2-IO36/A4)
- R2 pad 1: Net-(A2-I34/A2) -> GND
- R2 pad 2: GND -> Net-(A2-IO36/A4)
- R3 pad 2: Net-(A2-A8/IO15) -> Net-(A2-A10/IO27)
- R5 pad 2: Net-(A2-A10/IO27) -> Net-(A2-A8/IO15)
- R6 pad 1: SCL -> +3.3V
- R6 pad 2: +3.3V -> SCL
- TP1 pad 1: Net-(U2-ELE1) -> Net-(U3-ELE1)
- TP2 pad 1: Net-(U2-ELE2) -> Net-(U3-ELE2)
- TP3 pad 1: Net-(U2-ELE3) -> Net-(U3-ELE3)
- TP4 pad 1: Net-(U2-LED0/ELE4) -> Net-(U3-LED0/ELE4)
- TP5 pad 1: Net-(U2-LED1/ELE5) -> Net-(U3-LED1/ELE5)
- TP6 pad 1: Net-(U2-LED2/ELE6) -> Net-(U3-LED2/ELE6)
- TP7 pad 1: Net-(U2-LED3/ELE7) -> Net-(U3-LED3/ELE7)
- TP8 pad 1: Net-(U2-LED4/ELE8) -> Net-(U3-LED4/ELE8)
- U1 pad 3: Net-(A2-IO36/A4) -> Net-(A2-I39/A3)
- U2 pad 11: Net-(U2-ELE3) -> unconnected-(U2-~{RST}-Pad11)
- U2 pad 14: Net-(U2-LED2/ELE6) -> unconnected-(U2-INT-Pad14)
- U2 pad 19: unconnected-(U2-LED7/ELE11-Pad19) -> SCL
- U2 pad 2: SCL -> GND
- U2 pad 20: +3.3V -> SDA
- U2 pad 3: SDA -> +3.3V
- U2 pad 4: unconnected-(U2-ADDR-Pad4) -> +3.3V
- U2 pad 5: +3.3V -> unconnected-(U2-PS1-Pad5)
- U2 pad 6: GND -> unconnected-(U2-PS0-Pad6)
- U3 pad 11: unconnected-(U3-~{RST}-Pad11) -> Net-(U3-ELE3)
- U3 pad 14: unconnected-(U3-INT-Pad14) -> Net-(U3-LED2/ELE6)
- U3 pad 19: SCL -> unconnected-(U3-LED7/ELE11-Pad19)
- U3 pad 2: GND -> SCL
- U3 pad 20: SDA -> +3.3V
- U3 pad 3: +3.3V -> SDA
- U3 pad 4: +3.3V -> unconnected-(U3-ADDR-Pad4)
- U3 pad 5: unconnected-(U3-PS1-Pad5) -> +3.3V
Routing:
- net SCL: track 0.00 -> 178.9 mm
- net SDA: track 0.00 -> 177.7 mm
- net Net-(A2-I39/A3): track 0.00 -> 45.5 mm
- net Net-(A2-EN): track 0.00 -> 44.6 mm
- net Net-(U3-LED4/ELE8): track 0.00 -> 36.0 mm
- net Net-(U3-ELE1): track 0.00 -> 34.8 mm
- net Net-(A2-A10/IO27): track 0.00 -> 34.5 mm
- net Net-(A2-I34/A2): track 0.00 -> 32.8 mm
- net Net-(A2-A9/IO33): track 0.00 -> 32.1 mm
- net Net-(A2-A8/IO15): track 0.00 -> 30.7 mm
- net Net-(U3-LED3/ELE7): track 0.00 -> 28.2 mm
- net Net-(U3-ELE2): track 0.00 -> 27.0 mm
- net GND: track 0.00 -> 22.8 mm
- net Net-(A2-IO36/A4): track 0.00 -> 22.1 mm
- net Net-(U3-LED2/ELE6): track 0.00 -> 21.2 mm
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Other:
- outline, holes or cut-outs redrawn
- copper layers 2 -> 4
- board text added: "02/2025 - v1.0"
- board text removed: "v1.0"

Commit message: updates
Parts:
- moved LED 6.23 mm to (129.1, 62.1)
- moved R3 6.23 mm to (122.8, 54.7)
- moved R4 6.23 mm to (122.8, 58.7)
- moved R5 6.23 mm to (122.9, 62.7)
- moved H6 2.52 mm to (144.3, 85.4)
- moved H5 2.52 mm to (113.8, 85.4)
- moved B1 0.53 mm to (79.6, 75.2)
- renumbered D1 to LED, SW1 to POWER
Routing:
- net Net-(A2-A8/IO15): track 30.7 -> 28.2 mm
- net Net-(A2-A9/IO33): track 32.1 -> 29.6 mm
- net Net-(A2-A10/IO27): track 34.5 -> 32.0 mm
Changed lines of the file:
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@@
 			(drillshape 0)
 			(scaleselection 1)
-			(outputdirectory "gerbers/")
+			(outputdirectory "tesi-gerbers/")
 		)
 	)
@@
 	(footprint "Resistor_THT:R_Axial_DIN0207_L6.3mm_D2.5mm_P7.62mm_Horizontal"
 		(layer "F.Cu")
-		(at 129.043759 58.829548 180)
+		(at 122.81 58.744314 180)
 		(descr "Resistor, Axial_DIN0207 series, Axial, Horizontal, pin pitch=7.62mm, 0.25W = 1/4W, length*diameter=6.3*2.5mm^2, http://cdn-reichelt.de/documents/datenblatt/B400/1_4W%23YAG.pdf")
 		(tags "Resistor Axial_DIN0207 series Axial Horizontal pin pitch 7.62mm 0.25W = 1/4W length 6.3mm diameter 2.5mm")
@@
 		(tags " Adafruit Feather M0 RFM")
 		(property "Reference" "A2"
-			(at 9.5 47.25 180)
+			(at 9.667841 16.6195 180)
 			(layer "F.SilkS")
 			(hide yes)
@@
 		)
 		(property "Value" "ESP32"
-			(at 10.0525 19.05 180)
+			(at 9.917841 18.8695 0)
 			(layer "F.SilkS")
 			(effects
@@
 		(fp_line
 			(start 6 -6.5)
-			(end 6 2)
+			(end 6 -2.25)
 			(stroke
 				(width 0.1)
@@
 		)
 		(fp_line
-			(start 6 2)
-			(end 14.5 2)
+			(start 6 -2.25)
+			(end 14.5 -2.25)
 			(stroke
 				(width 0.1)
@@
 		)
 		(fp_line
-			(start 14.5 2)
+			(start 14.5 -2.25)
 			(end 14.5 -6.5)
 			(stroke
@@
 		)
 		(fp_line
-			(start 17 0.25)
-			(end 21.5 0.25)
-			(stroke
-				(width 0.1)
-				(type default)
-			)
-			(layer "F.SilkS")
-		)
-		(fp_line
-			(start 17 6)
-			(end 17 0.25)
-			(stroke
-				(width 0.1)
-				(type default)
-			)
-			(layer "F.SilkS")
-		)
-		(fp_line
 			(start 19.05 -6.46)
 			(end 1.27 -6.46)
@@
 		)
 		(fp_line
-			(start 21.5 6)
-			(end 17 6)
-			(stroke
-				(width 0.1)
-				(type default)
-			)
-			(layer "F.SilkS")
-		)
-		(fp_line
 			(start 21.7 -3.81)
 			(end 21.7 41.91)
@@
 			)
 		)
-		(fp_text user "BAT"
-			(at 20 4.5 90)
-			(unlocked yes)
-			(layer "F.SilkS")
-			(effects
-				(font
-					(size 1 1)
-					(thickness 0.1)
-				)
-				(justify left bottom)
-			)
-		)
 		(fp_text user "EN"
 			(at 15.4 13.3 0)
@@
 			)
 		)
-		(fp_text user "USB"
-			(at 8.667841 -1.6305 0)
-			(unlocked yes)
-			(layer "F.SilkS")
-			(effects
-				(font
-					(size 1 1)
-					(thickness 0.1)
-				)
-				(justify left bottom)
-			)
-		)
 		(fp_text user "MO"
 			(at 1.9 28.5 0)
@@
 			(at 1.718241 1.47 0)
 			(layer "F.SilkS")
+			(hide yes)
 			(effects
 				(font
@@
 			(at 30.364259 16.8186 0)
 			(layer "F.SilkS")
+			(hide yes)
 			(effects
 				(font
@@
 			(at 1.380941 1.18 180)
 			(layer "F.SilkS")
+			(hide yes)
 			(effects
 				(font
@@
 	(footprint "tesi:MountingHole_3.2mm_M3"
 		(layer "F.Cu")
-		(at 113.808332 87.926886)
+		(at 113.80344 85.411602)
 		(descr "Mounting Hole 3.2mm, no annular, M3")
 		(tags "mounting hole 3.2mm no annular m3")
@@
 	(footprint "Resistor_THT:R_Axial_DIN0207_L6.3mm_D2.5mm_P7.62mm_Horizontal"
 		(layer "F.Cu")
-		(at 129.103759 62.829548 180)
+		(at 122.87 62.744314 180)
 		(descr "Resistor, Axial_DIN0207 series, Axial, Horizontal, pin pitch=7.62mm, 0.25W = 1/4W, length*diameter=6.3*2.5mm^2, http://cdn-reichelt.de/documents/datenblatt/B400/1_4W%23YAG.pdf")
 		(tags "Resistor Axial_DIN0207 series Axial Horizontal pin pitch 7.62mm 0.25W = 1/4W length 6.3mm diameter 2.5mm")
@@
 		(descr "CuK miniature slide switch, OS series, SPDT, right angle, http://www.ckswitches.com/media/1428/os.pdf")
 		(tags "switch SPDT")
-		(property "Reference" "SW1"
-			(at 1.8 4.75 180)
+		(property "Reference" "POWER"
+			(at 1.923759 4.75 180)
 			(layer "F.SilkS")
 			(effects
@@
 			(unlocked yes)
 			(layer "F.SilkS")
+			(hide yes)
 			(effects
 				(font
@@
 			(unlocked yes)
 			(layer "F.SilkS")
+			(hide yes)
 			(effects
 				(font
@@
 				(font
 					(size 1 1)
-					(thickness 0.125)
+					(thickness 0.15)
 				)
 			)
@@
 	(footprint "LED_THT:LED_D5.0mm-4_RGB_Wide_Pins"
 		(layer "F.Cu")
-		(at 135.292478 62.159 90)
+		(at 129.058719 62.073766 90)
 		(descr "LED, diameter 5.0mm, 4 pins, WP154A4, https://www.kingbright.com/attachments/file/psearch/000/00/00/L-154A4SUREQBFZGEW(Ver.11A).pdf")
 		(tags "LED diameter 5.0mm 2 pins diameter 5.0mm 3 pins diameter 5.0mm 4 pins RGB RGBLED")
-		(property "Reference" "D1"
-			(at 3.2385 -3.96 90)
+		(property "Reference" "LED"
+			(at 3.242336 5.941281 180)
 			(layer "F.SilkS")
 			(hide yes)
@@
 	(footprint "Button_Switch_THT:SW_PUSH_6mm"
 		(layer "F.Cu")
-		(at 79.623759 75.7 180)
+		(at 79.623759 75.172691 180)
 		(descr "Generic 6mm SW tactile push button")
 		(tags "tact sw push 6mm")
@@
 	(footprint "tesi:MountingHole_3.2mm_M3"
 		(layer "F.Cu")
-		(at 144.327193 87.955978)
+		(at 144.322301 85.440694)
 		(descr "Mounting Hole 3.2mm, no annular, M3")
 		(tags "mounting hole 3.2mm no annular m3")
@@
 	(footprint "Resistor_THT:R_Axial_DIN0207_L6.3mm_D2.5mm_P7.62mm_Horizontal"
 		(layer "F.Cu")
-		(at 129.043759 54.829548 180)
+		(at 122.81 54.744314 180)
 		(descr "Resistor, Axial_DIN0207 series, Axial, Horizontal, pin pitch=7.62mm, 0.25W = 1/4W, length*diameter=6.3*2.5mm^2, http://cdn-reichelt.de/documents/datenblatt/B400/1_4W%23YAG.pdf")
 		(tags "Resistor Axial_DIN0207 series Axial Horizontal pin pitch 7.62mm 0.25W = 1/4W length 6.3mm diameter 2.5mm")
@@
 	)
 	(segment
-		(start 120.233759 73.6989)
-		(end 120.233759 60.019548)
+		(start 112.127 81.805659)
+		(end 108.402159 85.5305)
 		(width 0.5)
 		(layer "B.Cu")
@@
 	)
 	(segment
-		(start 120.233759 60.019548)
-		(end 121.423759 58.829548)
+		(start 115.19 58.744314)
+		(end 112.127 61.807314)
 		(width 0.5)
 		(layer "B.Cu")
@@
 	)
 	(segment
-		(start 108.402159 85.5305)
-		(end 120.233759 73.6989)
+		(start 112.127 61.807314)
+		(end 112.127 81.805659)
 		(width 0.5)
 		(layer "B.Cu")
@@
 	)
 	(segment
-		(start 109.923759 86.5489)
-		(end 108.402159 88.0705)
+		(start 110.5 84.319371)
+		(end 110.5 85.972659)
 		(width 0.5)
 		(layer "B.Cu")
@@
 	)
 	(segment
-		(start 121.483759 62.829548)
-		(end 120.933759 63.379548)
+		(start 115.25 62.744314)
+		(end 112.754 65.240314)
 		(width 0.5)
 		(layer "B.Cu")
@@
 	)
 	(segment
-		(start 120.933759 73.98885)
-		(end 109.923759 84.99885)
+		(start 112.754 82.065371)
+		(end 110.5 84.319371)
 		(width 0.5)
 		(layer "B.Cu")
@@
 	)
 	(segment
-		(start 109.923759 84.99885)
-		(end 109.923759 86.5489)
+		(start 112.754 65.240314)
+		(end 112.754 82.065371)
 		(width 0.5)
 		(layer "B.Cu")
@@
 	)
 	(segment
-		(start 120.933759 63.379548)
-		(end 120.933759 73.98885)
+		(start 110.5 85.972659)
+		(end 108.402159 88.0705)
 		(width 0.5)
 		(layer "B.Cu")
@@
 	)
 	(segment
-		(start 109.952209 82.9905)
+		(start 108.401759 82.9905)
 		(end 108.402159 82.9905)
 		(width 0.5)
@@
 	)
 	(segment
-		(start 119.473759 56.779548)
-		(end 119.473759 73.46895)
+		(start 111.5 81.545947)
+		(end 110.055447 82.9905)
 		(width 0.5)
 		(layer "B.Cu")
@@
 	)
 	(segment
-		(start 119.473759 73.46895)
-		(end 109.952209 82.9905)
+		(start 115.19 54.744314)
+		(end 111.5 58.434314)
 		(width 0.5)
 		(layer "B.Cu")
@@
 	)
 	(segment
-		(start 108.401759 82.9905)
-		(end 108.402159 82.9905)
+		(start 111.5 58.434314)
+		(end 111.5 81.545947)
 		(width 0.5)
 		(layer "B.Cu")
@@
 	)
 	(segment
-		(start 121.423759 54.829548)
-		(end 119.473759 56.779548)
+		(start 110.055447 82.9905)
+		(end 108.402159 82.9905)
 		(width 0.5)
 		(layer "B.Cu")
@@
 	)
 	(segment
-		(start 131.933307 60)
-		(end 129.103759 62.829548)
+		(start 125.699548 59.914766)
+		(end 122.87 62.744314)
 		(width 0.5)
 		(layer "B.Cu")
@@
 	)
 	(segment
-		(start 135.292478 60)
-		(end 131.933307 60)
+		(start 129.058719 59.914766)
+		(end 125.699548 59.914766)
 		(width 0.5)
 		(layer "B.Cu")
@@
 	)
 	(segment
-		(start 135.292478 55.682)
-		(end 129.896211 55.682)
+		(start 129.058719 55.596766)
+		(end 123.662452 55.596766)
 		(width 0.5)
 		(layer "B.Cu")
@@
 	)
 	(segment
-		(start 129.896211 55.682)
-		(end 129.043759 54.829548)
+		(start 123.662452 55.596766)
+		(end 122.81 54.744314)
 		(width 0.5)
 		(layer "B.Cu")
@@
 	)
 	(segment
-		(start 135.292478 57.841)
-		(end 130.032307 57.841)
+		(start 129.058719 57.755766)
+		(end 123.798548 57.755766)
 		(width 0.5)
 		(layer "B.Cu")
@@
 	)
 	(segment
-		(start 130.032307 57.841)
-		(end 129.043759 58.829548)
+		(start 123.798548 57.755766)
+		(end 122.81 58.744314)
 		(width 0.5)
 		(layer "B.Cu")
@@
 	)
 	(segment
-		(start 76.323759 60.9845)
-		(end 76.323759 60)
-		(width 0.5)
-		(layer "B.Cu")
-		(net 28)
-	)
-	(segment
-		(start 79.623759 75.7)
-		(end 79.223759 75.7)
+		(start 79.623759 75.172691)
+		(end 73.123759 75.172691)
 		(width 0.5)
 		(layer "B.Cu")
@@
 	)
 	(segment
-		(start 79.223759 75.7)
-		(end 79.173759 75.75)
+		(start 76.323759 60.9845)
+		(end 76.323759 60)
 		(width 0.5)
 		(layer "B.Cu")
@@
 	)
 	(segment
-		(start 79.173759 75.75)
-		(end 79.123759 75.7)
-		(width 0.5)
-		(layer "B.Cu")
-		(net 28)
-	)
-	(segment
 		(start 76.2695 60.2305)
 		(end 76.25 60.25)
@@
 	)
 	(segment
-		(start 79.123759 75.7)
-		(end 73.123759 75.7)
-		(width 0.5)
-		(layer "B.Cu")
-		(net 28)
-	)
-	(segment
 		(start 108.552759 93)
 		(end 108.401759 93.1505)
@@
 	)
 	(segment
-		(start 84.873759 71.2)
-		(end 86.504259 72.8305)
-		(width 0.5)
-		(layer "B.Cu")
-		(net 32)
-	)
-	(segment
-		(start 79.623759 71.2)
-		(end 84.873759 71.2)
+		(start 73.123759 70.672691)
+		(end 79.623759 70.672691)
 		(width 0.5)
 		(layer "B.Cu")
@@
 	)
 	(segment
-		(start 73.123759 71.2)
-		(end 79.623759 71.2)
+		(start 81.781568 72.8305)
+		(end 79.623759 70.672691)
 		(width 0.5)
 		(layer "B.Cu")
@@
 	)
 	(segment
-		(start 86.504259 72.8305)
-		(end 88.082159 72.8305)
+		(start 88.082159 72.8305)
+		(end 81.781568 72.8305)
 		(width 0.5)
 		(layer "B.Cu")

Commit message: update pcb
Parts:
- added 3.3V: Conn_01x04_Pin, Connector_PinSocket_2.54mm:PinSocket_1x04_P2.54mm_Vertical, F.Cu at (54.0, 66.7)
- added GND: Conn_01x04_Pin, Connector_PinSocket_2.54mm:PinSocket_1x04_P2.54mm_Vertical, F.Cu at (60.2, 66.7)
- added J3: Conn_01x04_Pin, Connector_PinSocket_2.54mm:PinSocket_1x04_P2.54mm_Vertical, F.Cu at (53.3, 83.9)
- A2: value ESP32 -> Adafruit ESP32 Feather
- SW1: renamed from POWER; footprint Button_Switch_THT:SW_Slide_SPDT_Angled_CK_OS102011MA1Q -> Button_Switch_THT:SW_Slide_SPDT_Straight_CK_OS102011MS2Q
- moved B1 74.4 mm to (142.8, 114.5)
- moved R6 58.8 mm to (130.9, 110.2), turned to 180 degrees
- moved R7 55.3 mm to (130.9, 114.5), turned to 180 degrees
- moved SW1 38.1 mm to (116.3, 57.0), turned to -90 degrees
- moved R2 22.3 mm to (60.9, 102.8)
- moved R1 21.9 mm to (55.7, 95.8)
- moved VL53L1X 18.9 mm to (132.9, 125.5)
- moved MPR121 17.4 mm to (99.0, 120.7), turned to 0 degrees
- moved RV1 14.9 mm to (71.4, 76.5)
- moved U1 13.2 mm to (72.1, 92.6)
- moved D1 8.44 mm to (137.5, 62.2)
- moved R3 7.78 mm to (130.6, 54.5)
- moved R4 7.77 mm to (130.6, 58.8)
- moved R5 7.72 mm to (130.6, 63.0)
- moved U2 0.60 mm to (52.4, 110.2)
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- renumbered LED to D1, U3 to MPR121, U4 to VL53L1X
Connections:
- A2 pad 19: unconnected-(A2-A6/IO14-Pad19) -> Net-(A2-A6/IO14)
- A2 pad 20: unconnected-(A2-A7/IO32-Pad20) -> Net-(A2-A7/IO32)
Routing:
- net SCL: track 178.9 -> 0.00 mm
- net SDA: track 177.7 -> 0.00 mm
- net Net-(A2-I39/A3): track 45.5 -> 0.00 mm
- net Net-(A2-EN): track 44.6 -> 0.00 mm
- net Net-(U3-LED4/ELE8): track 36.0 -> 0.00 mm
- net Net-(U3-ELE1): track 34.8 -> 0.00 mm
- net Net-(A2-I34/A2): track 32.8 -> 0.00 mm
- net Net-(A2-A10/IO27): track 32.0 -> 0.00 mm
- net Net-(A2-A9/IO33): track 29.6 -> 0.00 mm
- net Net-(U3-LED3/ELE7): track 28.2 -> 0.00 mm
- net Net-(A2-A8/IO15): track 28.2 -> 0.00 mm
- net Net-(U3-ELE2): track 27.0 -> 0.00 mm
- net GND: track 22.8 -> 0.00 mm
- net Net-(A2-IO36/A4): track 22.1 -> 0.00 mm
- net Net-(U3-LED2/ELE6): track 21.2 -> 0.00 mm
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Other:
- board text added: "A6"
- board text added: "A7"
- board text added: "ID:"
- board text added: "SCL"
- board text added: "SDA"

Commit message: update pcb
Parts:
- removed BT1: LIPO BATTERY, tesi:Lipo Battery 500 mAh - 38x30.5mm
- added J4: Conn_01x04_Pin, Connector_PinSocket_2.54mm:PinSocket_1x04_P2.54mm_Vertical, F.Cu at (119.8, 107.3)
- added REF**: Perfboard_10x10, tesi:Perfboard_10x10, F.Cu at (48.6, 31.1)
- A2: value Adafruit ESP32 Feather -> Adafruit Feather HUZZAH32; footprint tesi:Adafruit HUZZAH32 Feather Board - WithoutMountingHoles -> tesi:Adafruit ESP32 Feather
- moved B1 96.2 mm to (74.6, 46.6), turned to 0 degrees
- moved R1 41.4 mm to (79.1, 61.6), turned to 180 degrees
- moved R2 38.4 mm to (74.0, 66.7), turned to 0 degrees
- moved R5 28.3 mm to (122.3, 36.0)
- moved SW1 28.0 mm to (137.9, 39.2)
- moved D1 26.2 mm to (127.4, 38.0), turned to -90 degrees
- moved U4 23.8 mm to (141.5, 103.3), turned to -90 degrees
- moved RV1 23.7 mm to (58.8, 56.5)
- moved +3.3V 21.4 mm to (74.0, 74.3), turned to 90 degrees
- moved U1 21.3 mm to (61.3, 74.3)
- moved J3 20.7 mm to (74.0, 84.4)
- moved R4 19.5 mm to (122.3, 41.1)
- moved GND 18.7 mm to (74.0, 79.3), turned to 90 degrees
- moved A2 18.6 mm to (89.2, 41.2)
- moved H3 18.5 mm to (54.6, 37.2)
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- renumbered 3.3V to +3.3V, MPR121 to U3, VL53L1X to U4
Connections:
- A2 pad 5: unconnected-(A2-DAC2/A0-Pad5) -> Net-(A2-DAC2/A0)
- A2 pad 9: Net-(A2-IO36/A4) -> unconnected-(A2-IO36/A4-Pad9)
- B1 pad 2: Net-(A2-DAC1/A1) -> Net-(A2-DAC2/A0)
- J3 pad 1: Net-(A2-A6/IO14) -> SDA
- J3 pad 2: Net-(A2-A7/IO32) -> SCL
- J3 pad 3: SCL -> Net-(A2-A7/IO32)
- J3 pad 4: SDA -> Net-(A2-A6/IO14)
- R1 pad 1: Net-(A2-IO36/A4) -> Net-(A2-I39/A3)
- R2 pad 2: Net-(A2-IO36/A4) -> Net-(A2-I39/A3)
- RV1 pad 2: Net-(A2-I34/A2) -> Net-(A2-DAC1/A1)
- TP1 pad 1: Net-(U3-ELE1) -> Net-(U3-ELE2)
- TP2 pad 1: Net-(U3-ELE2) -> Net-(U3-ELE3)
- TP3 pad 1: Net-(U3-ELE3) -> Net-(U3-LED0/ELE4)
- TP4 pad 1: Net-(U3-LED0/ELE4) -> Net-(U3-LED1/ELE5)
- TP5 pad 1: Net-(U3-LED1/ELE5) -> Net-(U3-LED2/ELE6)
- TP6 pad 1: Net-(U3-LED2/ELE6) -> Net-(U3-LED3/ELE7)
- TP7 pad 1: Net-(U3-LED3/ELE7) -> Net-(U3-LED4/ELE8)
- TP8 pad 1: Net-(U3-LED4/ELE8) -> Net-(U3-LED5/ELE9)
- U1 pad 3: Net-(A2-I39/A3) -> Net-(A2-I34/A2)
- U2 pad 4: +3.3V -> unconnected-(U2-3V-Pad4)
- U3 pad 17: unconnected-(U3-LED5/ELE9-Pad17) -> Net-(U3-LED5/ELE9)
- U3 pad 18: unconnected-(U3-LED6/ELE10-Pad18) -> Net-(J4-Pin_3)
- U3 pad 19: unconnected-(U3-LED7/ELE11-Pad19) -> Net-(J4-Pin_4)
- U3 pad 2: SCL -> unconnected-(U3-ADDR-Pad2)
- U3 pad 4: unconnected-(U3-ADDR-Pad4) -> SCL
- U3 pad 5: +3.3V -> unconnected-(U3-IRQ-Pad5)
- U3 pad 6: unconnected-(U3-GND-Pad6) -> +3.3V
- U3 pad 8: unconnected-(U3-ELE0-Pad8) -> Net-(J4-Pin_1)
- U3 pad 9: Net-(U3-ELE1) -> Net-(J4-Pin_2)
Routing:
- net SDA: track 0.00 -> 147.3 mm
- net SCL: track 0.00 -> 141.1 mm
- net Net-(A2-I34/A2): track 0.00 -> 49.7 mm
- net Net-(A2-A8/IO15): track 0.00 -> 49.0 mm
- net Net-(A2-A9/IO33): track 0.00 -> 40.1 mm
- net Net-(J4-Pin_2): track 0.00 -> 37.2 mm
- net Net-(J4-Pin_1): track 0.00 -> 36.5 mm
- net Net-(A2-A7/IO32): track 0.00 -> 35.7 mm
- net Net-(U3-LED5/ELE9): track 0.00 -> 34.6 mm
- net Net-(U3-ELE2): track 0.00 -> 34.6 mm
- net Net-(A2-EN): track 0.00 -> 32.8 mm
- net Net-(A2-A6/IO14): track 0.00 -> 32.1 mm
- net Net-(A2-A10/IO27): track 0.00 -> 30.1 mm
- net Net-(A2-DAC1/A1): track 0.00 -> 29.0 mm
- net Net-(U3-LED4/ELE8): track 0.00 -> 26.0 mm
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Other:
- copper layers 4 -> 2
- board text added: "0"
- board text added: "1"
- board text added: "10"
- board text added: "11"
- board text added: "A6/14"
- board text added: "A7/32"
- board text added: "Adafruit ESP32 Feather"
- board text added: "MPR121"
- board text added: "VL53L1X"
- board text removed: "A6"
- board text removed: "A7"

Commit message: update pcb
Parts:
- removed +3.3V, GND: Conn_01x04_Pin, Connector_PinSocket_2.54mm:PinSocket_1x04_P2.54mm_Vertical
- added J1: Conn_01x03_Pin, Connector_PinSocket_2.54mm:PinSocket_1x03_P2.54mm_Vertical, F.Cu at (75.3, 74.2)
- added J2: Conn_01x03_Pin, Connector_PinSocket_2.54mm:PinSocket_1x03_P2.54mm_Vertical, F.Cu at (75.3, 79.3)
- moved J4 2.48 mm to (122.2, 107.2)
- moved R6 2.48 mm to (129.9, 97.0)
- moved R7 2.48 mm to (129.9, 102.1)
- moved J3 1.26 mm to (75.3, 84.3)
Connections:
- A2 pad 10: unconnected-(A2-IO4/A5-Pad10) -> Net-(A2-IO4/A5)
- A2 pad 19: Net-(A2-A6/IO14) -> unconnected-(A2-A6/IO14-Pad19)
- A2 pad 20: Net-(A2-A7/IO32) -> unconnected-(A2-A7/IO32-Pad20)
- A2 pad 9: unconnected-(A2-IO36/A4-Pad9) -> Net-(A2-IO36/A4)
- J3 pad 1: SDA -> GND
- J3 pad 2: SCL -> +3.3V
- J3 pad 3: Net-(A2-A7/IO32) -> SDA
- J3 pad 4: Net-(A2-A6/IO14) -> SCL
Routing:
- net Net-(A2-A7/IO32): track 35.7 -> 0.00 mm
- net Net-(A2-A6/IO14): track 32.1 -> 0.00 mm
- net Net-(A2-IO4/A5): track 0.00 -> 20.8 mm
- net Net-(A2-IO36/A4): track 0.00 -> 18.7 mm
- net SCL: track 141.1 -> 134.9 mm
- net SDA: track 147.3 -> 141.5 mm
- net Net-(J4-Pin_3): track 15.9 -> 18.6 mm
- net Net-(J4-Pin_4): track 16.3 -> 18.9 mm
- net Net-(J4-Pin_1): track 36.5 -> 39.0 mm
- net Net-(J4-Pin_2): track 37.2 -> 39.6 mm
Other:
- board text added: "3V"
- board text added: "A6"
- board text added: "A7"
- board text added: "GND"
- board text removed: "A6/14"
- board text removed: "A7/32"

Commit message: updates
Parts:
- removed REF**: Perfboard_10x10, tesi:Perfboard_10x10
- moved SW1 0.06 mm to (137.8, 39.2)
Routing:
- net SCL: track 134.9 -> 132.6 mm
Other:
- board text added: "POWER"
