File: kicad/tesi.kicad_pcb (KiCad board)
At the start: 2 copper layers, 100 x 100 mm, 34 parts, among them J1 Conn_01x03_Pin, J2 Conn_01x03_Pin, J3 Conn_01x04_Pin, J4 Conn_01x04_Pin, SW1 POWER, U1 MAX4466, U2 BNO055, U3 MPR121, U4 VL53L1CX

Commit message: updates
Parts:
- added C1: C_Polarized, tesi:CP_Radial_D4.0mm_P2.00mm, F.Cu at (77.0, 38.0)
- J4: value Conn_01x04_Pin -> Conn_01x02_Pin; footprint Connector_PinSocket_2.54mm:PinSocket_1x04_P2.54mm_Vertical -> Connector_PinSocket_2.54mm:PinSocket_1x02_P2.54mm_Vertical
- R2, R3, R4, R5: footprint Resistor_THT:R_Axial_DIN0207_L6.3mm_D2.5mm_P7.62mm_Horizontal -> Resistor_THT:R_Axial_DIN0207_L6.3mm_D2.5mm_P10.16mm_Horizontal
- R6: renamed from R7; footprint Resistor_THT:R_Axial_DIN0207_L6.3mm_D2.5mm_P7.62mm_Horizontal -> Resistor_THT:R_Axial_DIN0207_L6.3mm_D2.5mm_P10.16mm_Horizontal
- R7: renamed from R6; footprint Resistor_THT:R_Axial_DIN0207_L6.3mm_D2.5mm_P7.62mm_Horizontal -> Resistor_THT:R_Axial_DIN0207_L6.3mm_D2.5mm_P10.16mm_Horizontal
- SW1: footprint Button_Switch_THT:SW_Slide_SPDT_Straight_CK_OS102011MS2Q -> tesi:Switch
- moved J3 62.9 mm to (137.8, 91.4)
- moved J4 39.7 mm to (86.8, 89.5)
- moved R2 22.9 mm to (71.8, 89.5)
- moved R1 21.2 mm to (78.2, 82.8)
- moved U2 16.3 mm to (66.9, 103.4)
- moved J2 14.8 mm to (74.5, 64.5)
- moved J1 13.3 mm to (74.5, 60.9)
- moved R6 11.1 mm to (132.9, 91.4)
- moved U4 8.14 mm to (134.1, 106.7), turned to 0 degrees
- moved RV1 4.41 mm to (58.7, 60.9)
- moved U1 3.93 mm to (61.3, 78.2)
- moved R5 3.81 mm to (125.0, 38.6)
- moved R7 3.68 mm to (132.9, 94.9)
- moved D1 3.39 mm to (130.7, 38.8)
- moved R3 2.99 mm to (125.0, 45.1)
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Connections:
- J1 pad 3: Net-(A2-IO36/A4) -> Net-(A2-I34/A2)
- J2 pad 3: Net-(A2-IO4/A5) -> Net-(A2-I39/A3)
- R1 pad 1: Net-(A2-I39/A3) -> Net-(A2-IO4/A5)
- R2 pad 2: Net-(A2-I39/A3) -> Net-(A2-IO4/A5)
- U1 pad 3: Net-(A2-I34/A2) -> Net-(A2-IO36/A4)
- U3 pad 18: Net-(J4-Pin_3) -> unconnected-(U3-LED6/ELE10-Pad18)
- U3 pad 19: Net-(J4-Pin_4) -> unconnected-(U3-LED7/ELE11-Pad19)
Routing:
- net SCL: track 132.6 -> 201.3 mm
- net Net-(A2-I34/A2): track 49.7 -> 11.4 mm
- net Net-(A2-IO36/A4): track 18.7 -> 42.4 mm
- net Net-(J4-Pin_4): track 18.9 -> 0.00 mm
- net Net-(J4-Pin_3): track 18.6 -> 0.00 mm
- net Net-(J4-Pin_2): track 39.6 -> 22.8 mm
- net Net-(J4-Pin_1): track 39.0 -> 22.8 mm
- net GND: track 0.00 -> 15.8 mm
- net +3.3V: track 0.00 -> 14.6 mm
- net SDA: track 141.5 -> 129.7 mm
- net Net-(A2-IO4/A5): track 20.8 -> 32.0 mm
- net Net-(A2-A8/IO15): track 49.0 -> 43.3 mm
- net Net-(A2-I39/A3): track 17.3 -> 11.9 mm
- net Net-(A2-A9/IO33): track 39.6 -> 35.7 mm
- net Net-(A2-DAC1/A1): track 29.0 -> 31.9 mm
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Other:
- board text added: "A3"
- board text added: "A4"
- board text added: "Designed at d.search lab – TU/e"
- board text removed: "0"
- board text removed: "1"
- board text removed: "10"
- board text removed: "11"
- board text removed: "A6"
- board text removed: "A7"
- board text removed: "MPR121"
- board text removed: "VL53L1X"

Commit message: updates
Parts:
- removed the J2 at (74.5, 64.5)
- removed J3: Conn_01x04_Pin, Connector_PinSocket_2.54mm:PinSocket_1x04_P2.54mm_Vertical
- added B2: ~, Button_Switch_THT:SW_PUSH_6mm, F.Cu at (81.0, 67.6)
- added C2: C, Capacitor_THT:C_Disc_D4.3mm_W1.9mm_P5.00mm, F.Cu at (80.4, 42.9)
- J1: renamed from J4; value Conn_01x02_Pin -> Conn_01x02_Socket
- J2: renamed from J1; value Conn_01x03_Pin -> Conn_01x06_Socket; footprint Connector_PinSocket_2.54mm:PinSocket_1x03_P2.54mm_Vertical -> Connector_PinSocket_2.54mm:PinSocket_1x06_P2.54mm_Vertical
- R2: value 5K -> 10K
- moved J2 64.2 mm to (132.0, 89.5)
- moved RV1 28.6 mm to (58.5, 89.5)
- moved R6 23.4 mm to (109.6, 89.5)
- moved U1 19.5 mm to (61.3, 58.7)
- moved B1 11.0 mm to (81.1, 55.2), turned to 180 degrees
- moved R7 9.92 mm to (124.6, 89.5)
- moved R3 8.00 mm to (124.6, 37.1)
- moved R5 4.48 mm to (124.6, 43.1)
- moved H5 2.60 mm to (115.7, 66.0)
- moved H6 2.60 mm to (146.6, 66.0)
- moved SW1 2.05 mm to (139.5, 38.1)
- moved D1 1.98 mm to (130.3, 36.9)
- moved C1 1.95 mm to (78.9, 37.2), turned to 180 degrees
- moved R4 1.80 mm to (124.6, 40.1)
- moved R1 1.25 mm to (79.1, 82.0)
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- renumbered A2 to A1
Connections:
- A1 pad 10: Net-(A2-IO4/A5) -> unconnected-(A1-IO4/A5-Pad10)
- A1 pad 19: unconnected-(A2-A6/IO14-Pad19) -> Net-(A1-A6/IO14)
- A1 pad 20: unconnected-(A2-A7/IO32-Pad20) -> Net-(A1-A7/IO32)
- A1 pad 21: Net-(A2-A8/IO15) -> Net-(A1-A8/IO15)
- A1 pad 22: Net-(A2-A9/IO33) -> Net-(A1-A9/IO33)
- A1 pad 23: Net-(A2-A10/IO27) -> Net-(A1-A10/IO27)
- A1 pad 6: Net-(A2-DAC1/A1) -> Net-(A1-DAC1/A1)
- A1 pad 7: Net-(A2-I34/A2) -> Net-(A1-I34/A2)
- A1 pad 8: Net-(A2-I39/A3) -> Net-(A1-I39/A3)
- A1 pad 9: Net-(A2-IO36/A4) -> Net-(A1-IO36/A4)
- D1 pad 1: +3.3V -> Net-(D1-RK)
- D1 pad 2: Net-(D1-RK) -> GND
- J2 pad 3: Net-(A2-I34/A2) -> SCL
- R1 pad 1: Net-(A2-IO4/A5) -> Net-(A1-IO36/A4)
- R2 pad 2: Net-(A2-IO4/A5) -> Net-(A1-IO36/A4)
- R3 pad 1: Net-(D1-BK) -> Net-(D1-RK)
- R3 pad 2: Net-(A2-A10/IO27) -> Net-(A1-A6/IO14)
- R4 pad 2: Net-(A2-A9/IO33) -> Net-(A1-A8/IO15)
- R5 pad 1: Net-(D1-RK) -> Net-(D1-BK)
- R5 pad 2: Net-(A2-A8/IO15) -> Net-(A1-A10/IO27)
- RV1 pad 2: Net-(A2-DAC1/A1) -> Net-(A1-I39/A3)
- U1 pad 3: Net-(A2-IO36/A4) -> Net-(A1-I34/A2)
Routing:
- net SCL: track 201.3 -> 133.2 mm
- net Net-(A1-A6/IO14): track 0.00 -> 53.4 mm
- net Net-(A1-I39/A3): track 0.00 -> 52.6 mm
- net Net-(A1-IO36/A4): track 0.00 -> 49.6 mm
- net Net-(A1-A9/IO33): track 0.00 -> 47.4 mm
- net Net-(A1-I34/A2): track 0.00 -> 44.4 mm
- net Net-(A2-A8/IO15): track 43.3 -> 0.00 mm
- net Net-(A2-IO36/A4): track 42.4 -> 0.00 mm
- net Net-(A1-A7/IO32): track 0.00 -> 42.3 mm
- net Net-(A1-A8/IO15): track 0.00 -> 41.9 mm
- net Net-(A2-A9/IO33): track 35.7 -> 0.00 mm
- net Net-(A2-IO4/A5): track 32.0 -> 0.00 mm
- net Net-(A2-DAC1/A1): track 31.9 -> 0.00 mm
- net Net-(A1-A10/IO27): track 0.00 -> 30.4 mm
- net Net-(A2-A10/IO27): track 28.2 -> 0.00 mm
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Other:
- board text added: "3.3V"
- board text added: "A7"
- board text added: "A9"
- board text removed: "3V"
- board text removed: "A3"
- board text removed: "A4"
