File: kicad/tesi.kicad_sch (KiCad schematic)
At the start: 29 parts, among them SW1 POWER, U121 MPR121, U2 BNO055, U3 VL53L1CX

Commit message: add files
Parts:
- A2: footprint Library:Adafruit HUZZAH32 Feather Board - WithoutMountingHoles -> tesi:Adafruit HUZZAH32 Feather Board - WithoutMountingHoles
- H1, H2, H3, H4: value MH-3.2mm -> 3.2mm; footprint MountingHole:MountingHole_3.2mm_M3 -> tesi:MountingHole_3.2mm_M3; symbol Mechanical:MountingHole_Pad -> Mechanical:MountingHole
- H5, H6: value MountingHole -> 3.2mm - Battery; footprint MountingHole:MountingHole_4mm -> tesi:MountingHole_3.2mm_M3
- U1: renamed from MAX4466; value Electret Mic -> MAX4466; footprint Library:MAX4466 -> tesi:MAX4466; symbol board_symbols:MAX4466 -> tesi:MAX4466
- U2: renamed from U121; footprint Library:MPR121 -> tesi:MPR121; symbol board_symbols:MPR121 -> tesi:MPR121
- U3: renamed from U2; footprint Library:BNO055 -> tesi:BNO055; symbol board_symbols:BNO055 -> tesi:BNO055
- U4: renamed from U3; footprint Library:VL53L1X -> tesi:VL53L1X; symbol board_symbols:VL53L1CX -> tesi:VL53L1CX
- renumbered R8 to R1
Connections:
- net GND: no longer H1.1, H2.1, H3.1, H4.1
- net at R5.2: now also A2.21 (A8/IO15); no longer A2.23 (A10/IO27)
- net at R3.2: now also A2.23 (A10/IO27); no longer A2.21 (A8/IO15)
Other:
- title: (none) -> TESI
- moved on the sheet: H6

Commit message: updates
Parts:
- added BT1: Battery, tesi:Lipo Battery 500 mAh - 38x30.5mm, symbol Device:Battery
- added RV1: POT, Potentiometer_THT:Potentiometer_TT_P0915N, symbol Device:R_Potentiometer
- B1: value MUTE -> ~
- TP1, TP2, TP3, TP4, TP5, TP6, TP7, TP8: footprint TestPoint:TestPoint_Pad_D4.0mm -> tesi:TouchPad - 4.0mm
- renumbered R7 to R6, R6 to R7, U3 to U2, U2 to U3
Connections:
- net +3.3V: now also R6.1, RV1.3; no longer R6.2
- net GND: now also R2.1, RV1.1; no longer R2.2, U3.6 (GND)
- net SCL: now also R6.2; no longer R6.1
- net at U1.3 (OUT): now also A2.8 (I39/A3); no longer A2.9 (IO36/A4)
- net at B1.2: now also A2.6 (DAC1/A1); no longer A2.20 (A7/IO32)
- new net: A2.7 (I34/A2), RV1.2
- new net: A2.9 (IO36/A4), R1.1, R2.2
- no-connect marks 30 -> 32
Other:
- moved on the sheet: B1, R1, R2, R6

Commit message: update pcb
Parts:
- added J1, J2, J3: Conn_01x04_Pin, Connector_PinSocket_2.54mm:PinSocket_1x04_P2.54mm_Vertical, symbol Connector:Conn_01x04_Pin
- SW1: footprint Button_Switch_THT:SW_Slide_SPDT_Angled_CK_OS102011MA1Q -> Button_Switch_THT:SW_Slide_SPDT_Straight_CK_OS102011MS2Q
Connections:
- net +3.3V: now also J1.1 (Pin_1), J1.2 (Pin_2), J1.3 (Pin_3), J1.4 (Pin_4)
- net GND: now also J2.1 (Pin_1), J2.2 (Pin_2), J2.3 (Pin_3), J2.4 (Pin_4)
- net SCL: now also J3.3 (Pin_3)
- net SDA: now also J3.4 (Pin_4)
- net at A2.19 (A6/IO14): now also J3.1 (Pin_1)
- net at A2.20 (A7/IO32): now also J3.2 (Pin_2)
- no-connect marks 32 -> 31
Other:
- moved on the sheet: BT1

Commit message: update pcb
Parts:
- removed BT1: Battery, tesi:Lipo Battery 500 mAh - 38x30.5mm, symbol Device:Battery
- added J4: Conn_01x04_Pin, Connector_PinSocket_2.54mm:PinSocket_1x04_P2.54mm_Vertical, symbol Connector:Conn_01x04_Pin
- A2: footprint tesi:Adafruit HUZZAH32 Feather Board - WithoutMountingHoles -> tesi:Adafruit ESP32 Feather
Connections:
- net +3.3V: now also U3.6 (3.3V); no longer U2.4 (3V), U3.20 (Vin), U3.5 (3Vo)
- net GND: now also U3.1 (GND); no longer U3.7 (GND)
- net SCL: now also J3.2 (Pin_2), U3.4 (SCL); no longer J3.3 (Pin_3), U3.2 (SCL)
- net SDA: now also J3.1 (Pin_1); no longer J3.4 (Pin_4)
- net at TP4.1: now also U3.13 (LED1/ELE5); no longer U3.12 (LED0/ELE4)
- net at RV1.2: now also A2.6 (DAC1/A1); no longer A2.7 (I34/A2)
- net at TP8.1: now also U3.17 (LED5/ELE9); no longer U3.16 (LED4/ELE8)
- net at A2.19 (A6/IO14): now also J3.4 (Pin_4); no longer J3.1 (Pin_1)
- net at A2.20 (A7/IO32): now also J3.3 (Pin_3); no longer J3.2 (Pin_2)
- net at TP7.1: now also U3.16 (LED4/ELE8); no longer U3.15 (LED3/ELE7)
- net at U1.3 (OUT): now also A2.7 (I34/A2); no longer A2.8 (I39/A3)
- net at TP2.1: now also U3.11 (ELE3); no longer U3.10 (ELE2)
- net at TP6.1: now also U3.15 (LED3/ELE7); no longer U3.14 (LED2/ELE6)
- net at B1.2: now also A2.5 (DAC2/A0); no longer A2.6 (DAC1/A1)
- net at TP5.1: now also U3.14 (LED2/ELE6); no longer U3.13 (LED1/ELE5)
- net at R1.1, R2.2: now also A2.8 (I39/A3); no longer A2.9 (IO36/A4)
- net at U3.9 (ELE1): now also J4.2 (Pin_2); no longer TP1.1
- net at TP3.1: now also U3.12 (LED0/ELE4); no longer U3.11 (ELE3)
- net at U3.18 (LED6/ELE10): now also J4.3 (Pin_3)
- net at U3.19 (LED7/ELE11): now also J4.4 (Pin_4)
- net at U3.8 (ELE0): now also J4.1 (Pin_1)
- new net: TP1.1, U3.10 (ELE2)
- no-connect marks 31 -> 24
Other:
- moved on the sheet: B1, J3, R1, R2, SW1, TP1, TP2, TP3, TP4, TP5, TP6, TP7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

Commit message: update pcb
Parts:
- removed J1, J2: Conn_01x04_Pin, Connector_PinSocket_2.54mm:PinSocket_1x04_P2.54mm_Vertical, symbol Connector:Conn_01x04_Pin
- added J1, J2: Conn_01x03_Pin, Connector_PinSocket_2.54mm:PinSocket_1x03_P2.54mm_Vertical, symbol Connector:Conn_01x03_Pin
Connections:
- net +3.3V: now also J3.2 (Pin_2), J1.2 (Pin_2), J2.2 (Pin_2)
- net GND: now also J3.1 (Pin_1), J1.1 (Pin_1), J2.1 (Pin_1)
- net SCL: now also J3.4 (Pin_4); no longer J3.2 (Pin_2)
- net SDA: now also J3.3 (Pin_3); no longer J3.1 (Pin_1)
- net at A2.20 (A7/IO32): no longer J3.3 (Pin_3)
- net at A2.19 (A6/IO14): no longer J3.4 (Pin_4)
- net at A2.10 (IO4/A5): now also J2.3 (Pin_3)
- net at A2.9 (IO36/A4): now also J1.3 (Pin_3)
Other:
- moved on the sheet: J3

Commit message: updates
Parts:
- added C1: C_Polarized, tesi:CP_Radial_D4.0mm_P2.00mm, symbol Device:C_Polarized
- J4: value Conn_01x04_Pin -> Conn_01x02_Pin; footprint Connector_PinSocket_2.54mm:PinSocket_1x04_P2.54mm_Vertical -> Connector_PinSocket_2.54mm:PinSocket_1x02_P2.54mm_Vertical; symbol Connector:Conn_01x04_Pin -> Connector:Conn_01x02_Socket
- R2, R3, R4, R5: footprint Resistor_THT:R_Axial_DIN0207_L6.3mm_D2.5mm_P7.62mm_Horizontal -> Resistor_THT:R_Axial_DIN0207_L6.3mm_D2.5mm_P10.16mm_Horizontal
- R6: renamed from R7; footprint Resistor_THT:R_Axial_DIN0207_L6.3mm_D2.5mm_P7.62mm_Horizontal -> Resistor_THT:R_Axial_DIN0207_L6.3mm_D2.5mm_P10.16mm_Horizontal
- R7: renamed from R6; footprint Resistor_THT:R_Axial_DIN0207_L6.3mm_D2.5mm_P7.62mm_Horizontal -> Resistor_THT:R_Axial_DIN0207_L6.3mm_D2.5mm_P10.16mm_Horizontal
- SW1: footprint Button_Switch_THT:SW_Slide_SPDT_Straight_CK_OS102011MS2Q -> tesi:Switch
Connections:
- net +3.3V: now also C1.1
- net GND: now also C1.2
- net at U3.18 (LED6/ELE10): no longer J4.3 (Pin_3)
- net at U3.19 (LED7/ELE11): no longer J4.4 (Pin_4)
- net at J1.3 (Pin_3): now also A2.7 (I34/A2); no longer A2.9 (IO36/A4)
- net at U1.3 (OUT): now also A2.9 (IO36/A4); no longer A2.7 (I34/A2)
- net at R1.1, R2.2: now also A2.10 (IO4/A5); no longer A2.8 (I39/A3)
- net at J2.3 (Pin_3): now also A2.8 (I39/A3); no longer A2.10 (IO4/A5)
- no-connect marks 24 -> 26
Other:
- moved on the sheet: R1, R2

Commit message: updates
Parts:
- removed J1, J2: Conn_01x03_Pin, Connector_PinSocket_2.54mm:PinSocket_1x03_P2.54mm_Vertical, symbol Connector:Conn_01x03_Pin
- removed J3: Conn_01x04_Pin, Connector_PinSocket_2.54mm:PinSocket_1x04_P2.54mm_Vertical, symbol Connector:Conn_01x04_Pin
- added B2: ~, Button_Switch_THT:SW_PUSH_6mm, symbol Switch:SW_Push
- added C2: C, Capacitor_THT:C_Disc_D4.3mm_W1.9mm_P5.00mm, symbol Device:C
- added J2: Conn_01x06_Socket, Connector_PinSocket_2.54mm:PinSocket_1x06_P2.54mm_Vertical, symbol Connector:Conn_01x06_Socket
- D1: symbol Device:LED_ARGB -> tesi:RGB LED
- J1: renamed from J4; value Conn_01x02_Pin -> Conn_01x02_Socket
- R2: value 5K -> 10K
- renumbered A2 to A1, R5 to R3, R3 to R5
Connections:
- net +3.3V: now also C2.1, J2.2 (Pin_2); no longer D1.1 (A)
- net GND: now also D1.2 (A), B2.1, C2.2, J2.1 (Pin_1)
- net SCL: now also J2.3 (Pin_3)
- net SDA: now also J2.4 (Pin_4)
- net at A1.22 (A9/IO33): now also J2.6 (Pin_6); no longer R4.2
- net at A1.7 (I34/A2): now also U1.3 (OUT)
- net at RV1.2: now also A1.8 (I39/A3); no longer A1.6 (DAC1/A1)
- net at A1.9 (IO36/A4): now also R1.1, R2.2; no longer U1.3 (OUT)
- net at R3.1: now also D1.1 (RK); no longer D1.2 (RK)
- net at A1.21 (A8/IO15): now also R4.2; no longer R3.2
- net at A1.19 (A6/IO14): now also R3.2
- net at A1.20 (A7/IO32): now also J2.5 (Pin_5)
- new net: A1.6 (DAC1/A1), B2.2
- now unconnected: A1.10 (IO4/A5)
- no-connect marks 26 -> 25
Other:
- moved on the sheet: B1, C1, D1, J1, R1, R2, R3, R4, R5, SW1, TP1, TP2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
